Commit message: feat: add hu_d04 wbt climb_14 training support and gm-cli integration
- Add hu_d04 locomotion config values
- Add sim2sim scripts for hu_d04
- Add gm-cli skill for training platform integration
- Update simulator compatibility for isaacgym/isaacsim/mujoco
- Add bridge/sim2sim module

File: src/holosoma/holosoma/data/robots/hu_d04/hu_d04.urdf (robot description, URDF)
Before this commit: robot HU_D04_01, 42 links, 41 joints
Links:
- link base_link: geometry collision mesh filename=meshes/base_link.STL; visual mesh filename=meshes/base_link.STL
- link head_pitch_link: geometry collision mesh filename=meshes/neck_pitch_link.STL; visual mesh filename=meshes/neck_pitch_link.STL
- link head_yaw_link: geometry collision mesh filename=meshes/neck_yaw_link.STL; visual mesh filename=meshes/neck_yaw_link.STL
- link left_ankle_pitch_link: geometry collision mesh filename=meshes/left_ankle_pitch_link.STL; visual mesh filename=meshes/left_ankle_pitch_link.STL
- link left_ankle_roll_link: geometry collision box size=0.25 0.094 0.02; collision mesh filename=meshes/left_ankle_roll_link.STL
- link left_elbow_link: geometry collision mesh filename=meshes/left_elbow_link.STL; visual mesh filename=meshes/left_elbow_link.STL
- link left_hip_pitch_link: geometry collision mesh filename=meshes/left_hip_pitch_link.STL; visual mesh filename=meshes/left_hip_pitch_link.STL
- link left_hip_roll_link: geometry collision mesh filename=meshes/left_hip_roll_link.STL; visual mesh filename=meshes/left_hip_roll_link.STL
- link left_hip_yaw_link: geometry collision mesh filename=meshes/left_hip_yaw_link.STL; visual mesh filename=meshes/left_hip_yaw_link.STL
- link left_knee_link: geometry collision mesh filename=meshes/left_knee_link.STL; visual mesh filename=meshes/left_knee_link.STL
- link left_shoulder_pitch_link: geometry collision mesh filename=meshes/left_shoulder_pitch_link.STL; visual mesh filename=meshes/left_shoulder_pitch_link.STL
- link left_shoulder_roll_link: geometry collision mesh filename=meshes/left_shoulder_roll_link.STL; visual mesh filename=meshes/left_shoulder_roll_link.STL
- link left_shoulder_yaw_link: geometry collision mesh filename=meshes/left_shoulder_yaw_link.STL; visual mesh filename=meshes/left_shoulder_yaw_link.STL
- link left_wrist_pitch_link: geometry collision mesh filename=meshes/left_wrist_pitch_link.STL; visual mesh filename=meshes/left_wrist_pitch_link.STL
- link left_wrist_roll_link: geometry collision mesh filename=meshes/left_wrist_roll_link.STL; visual mesh filename=meshes/left_wrist_roll_link.STL
- link left_wrist_yaw_link: geometry collision mesh filename=meshes/left_wrist_yaw_link.STL; visual mesh filename=meshes/left_wrist_yaw_link.STL
- link right_ankle_pitch_link: geometry collision mesh filename=meshes/right_ankle_pitch_link.STL; visual mesh filename=meshes/right_ankle_pitch_link.STL
- link right_ankle_roll_link: geometry collision box size=0.25 0.094 0.02; collision mesh filename=meshes/right_ankle_roll_link.STL
- link right_elbow_link: geometry collision mesh filename=meshes/right_elbow_link.STL; visual mesh filename=meshes/right_elbow_link.STL
- link right_hip_pitch_link: geometry collision mesh filename=meshes/right_hip_pitch_link.STL; visual mesh filename=meshes/right_hip_pitch_link.STL
- link right_hip_roll_link: geometry collision mesh filename=meshes/right_hip_roll_link.STL; visual mesh filename=meshes/right_hip_roll_link.STL
- link right_hip_yaw_link: geometry collision mesh filename=meshes/right_hip_yaw_link.STL; visual mesh filename=meshes/right_hip_yaw_link.STL
- link right_knee_link: geometry collision mesh filename=meshes/right_knee_link.STL; visual mesh filename=meshes/right_knee_link.STL
- link right_shoulder_pitch_link: geometry collision mesh filename=meshes/right_shoulder_pitch_link.STL; visual mesh filename=meshes/right_shoulder_pitch_link.STL
- link right_shoulder_roll_link: geometry collision mesh filename=meshes/right_shoulder_roll_link.STL; visual mesh filename=meshes/right_shoulder_roll_link.STL
- link right_shoulder_yaw_link: geometry collision mesh filename=meshes/right_shoulder_yaw_link.STL; visual mesh filename=meshes/right_shoulder_yaw_link.STL
- link right_wrist_pitch_link: geometry collision mesh filename=meshes/right_wrist_pitch_link.STL; visual mesh filename=meshes/right_wrist_pitch_link.STL
- link right_wrist_roll_link: geometry collision mesh filename=meshes/right_wrist_roll_link.STL; visual mesh filename=meshes/right_wrist_roll_link.STL
- link right_wrist_yaw_link: geometry collision mesh filename=meshes/right_wrist_yaw_link.STL; visual mesh filename=meshes/right_wrist_yaw_link.STL
- link waist_pitch_link: geometry collision mesh filename=meshes/waist_pitch_link.STL; visual mesh filename=meshes/waist_pitch_link.STL
- link waist_roll_link: geometry collision mesh filename=meshes/waist_roll_link.STL; visual mesh filename=meshes/waist_roll_link.STL
- link waist_yaw_link: geometry collision mesh filename=meshes/waist_yaw_link.STL; visual mesh filename=meshes/waist_yaw_link.STL
Joints:
- joint head_pitch_joint: axis 0 1 0 -> (none); limit lower=-0.524 upper=0.785 effort=19 velocity=13 -> (none); type revolute -> fixed
- joint head_yaw_joint: axis 0 0 1 -> (none); limit lower=-0.785 upper=0.785 effort=19 velocity=13 -> (none); type revolute -> fixed
